File: fese75.kicad_pcb (KiCad board)
At the start: 2 copper layers, 4 parts

Commit message: quick place component
Parts:
- added '1: MX-NoLED, Switch_Keyboard_Kailh:SW_Hotswap_Kailh_1.00u, F.Cu at (215.0, -87.5)
- added +1: MX-NoLED, Switch_Keyboard_Kailh:SW_Hotswap_Kailh_1.00u, F.Cu at (219.0, -130.0)
- added ,1: MX-NoLED, Switch_Keyboard_Kailh:SW_Hotswap_Kailh_1.00u, F.Cu at (196.2, -66.8)
- added -1: MX-NoLED, Switch_Keyboard_Kailh:SW_Hotswap_Kailh_1.00u, F.Cu at (199.5, -129.8)
- added .1: MX-NoLED, Switch_Keyboard_Kailh:SW_Hotswap_Kailh_1.00u, F.Cu at (176.8, -67.0)
- added /1: MX-NoLED, Switch_Keyboard_Kailh:SW_Hotswap_Kailh_1.00u, F.Cu at (215.5, -67.2)
- added ;1: MX-NoLED, Switch_Keyboard_Kailh:SW_Hotswap_Kailh_1.00u, F.Cu at (196.0, -87.5)
- added A1: MX-NoLED, Switch_Keyboard_Kailh:SW_Hotswap_Kailh_1.00u, F.Cu at (24.0, -88.5)
- added ALT1: MX-NoLED, Switch_Keyboard_Kailh:SW_Hotswap_Kailh_1.00u, F.Cu at (36.5, -43.8)
- added ALT2: MX-NoLED, Switch_Keyboard_Kailh:SW_Hotswap_Kailh_1.00u, F.Cu at (175.8, -46.5)
- added B1: MX-NoLED, Switch_Keyboard_Kailh:SW_Hotswap_Kailh_1.00u, F.Cu at (112.5, -67.5)
- added BACK1: MX-NoLED, Switch_Keyboard_Kailh:SW_Hotswap_Kailh_1.00u, F.Cu at (251.5, -129.8)
- added C1: MX-NoLED, Switch_Keyboard_Kailh:SW_Hotswap_Kailh_1.00u, F.Cu at (64.2, -67.8)
- added CAPS1: MX-NoLED, Switch_Keyboard_Kailh:SW_Hotswap_Kailh_1.00u, F.Cu at (-4.25, -89.5)
- added CLT1: MX-NoLED, Switch_Keyboard_Kailh:SW_Hotswap_Kailh_1.00u, F.Cu at (-7.25, -44.5)
- added CTL1: MX-NoLED, Switch_Keyboard_Kailh:SW_Hotswap_Kailh_1.00u, F.Cu at (232.2, -45.2)
- added D1: D_Small, Diode_SMD:D_0603_1608Metric_Pad1.05x0.95mm_HandSolder, F.Cu at (-10.2, -157.2)
- added D10: D_Small, Diode_SMD:D_0603_1608Metric_Pad1.05x0.95mm_HandSolder, F.Cu at (177.5, -155.9)
- added D11: D_Small, Diode_SMD:D_0603_1608Metric_Pad1.05x0.95mm_HandSolder, F.Cu at (198.2, -156.0)
- added D12: D_Small, Diode_SMD:D_0603_1608Metric_Pad1.05x0.95mm_HandSolder, F.Cu at (218.2, -156.2)
- added D13: D_Small, Diode_SMD:D_0603_1608Metric_Pad1.05x0.95mm_HandSolder, F.Cu at (237.5, -155.6)
- added D14: D_Small, Diode_SMD:D_0603_1608Metric_Pad1.05x0.95mm_HandSolder, F.Cu at (266.5, -154.8)
- added D15: D_Small, Diode_SMD:D_0603_1608Metric_Pad1.05x0.95mm_HandSolder, F.Cu at (313.0, -158.0)
- added D16: D_Small, Diode_SMD:D_0603_1608Metric_Pad1.05x0.95mm_HandSolder, F.Cu at (-8.50, -123.2)
- added D17: D_Small, Diode_SMD:D_0603_1608Metric_Pad1.05x0.95mm_HandSolder, F.Cu at (10.0, -123.4)
- added D18: D_Small, Diode_SMD:D_0603_1608Metric_Pad1.05x0.95mm_HandSolder, F.Cu at (29.8, -124.0)
- added D19: D_Small, Diode_SMD:D_0603_1608Metric_Pad1.05x0.95mm_HandSolder, F.Cu at (48.8, -123.0)
- added D2: D_Small, Diode_SMD:D_0603_1608Metric_Pad1.05x0.95mm_HandSolder, F.Cu at (12.8, -158.1)
- added D20: D_Small, Diode_SMD:D_0603_1608Metric_Pad1.05x0.95mm_HandSolder, F.Cu at (69.2, -124.1)
- added D21: D_Small, Diode_SMD:D_0603_1608Metric_Pad1.05x0.95mm_HandSolder, F.Cu at (91.8, -124.2)
- added D22: D_Small, Diode_SMD:D_0603_1608Metric_Pad1.05x0.95mm_HandSolder, F.Cu at (111.2, -124.1)
- added D23: D_Small, Diode_SMD:D_0603_1608Metric_Pad1.05x0.95mm_HandSolder, F.Cu at (129.8, -124.5)
- added D24: D_Small, Diode_SMD:D_0603_1608Metric_Pad1.05x0.95mm_HandSolder, F.Cu at (149.8, -125.1)
- added D25: D_Small, Diode_SMD:D_0603_1608Metric_Pad1.05x0.95mm_HandSolder, F.Cu at (169.5, -125.0)
- added D26: D_Small, Diode_SMD:D_0603_1608Metric_Pad1.05x0.95mm_HandSolder, F.Cu at (187.5, -124.8)
- added D27: D_Small, Diode_SMD:D_0603_1608Metric_Pad1.05x0.95mm_HandSolder, F.Cu at (205.5, -124.4)
- added D28: D_Small, Diode_SMD:D_0603_1608Metric_Pad1.05x0.95mm_HandSolder, F.Cu at (224.0, -124.6)
- added D29: D_Small, Diode_SMD:D_0603_1608Metric_Pad1.05x0.95mm_HandSolder, F.Cu at (257.2, -124.2)
- added D3: D_Small, Diode_SMD:D_0603_1608Metric_Pad1.05x0.95mm_HandSolder, F.Cu at (32.2, -158.4)
- added D30: D_Small, Diode_SMD:D_0603_1608Metric_Pad1.05x0.95mm_HandSolder, F.Cu at (312.8, -125.6)
- added D31: D_Small, Diode_SMD:D_0603_1608Metric_Pad1.05x0.95mm_HandSolder, F.Cu at (0.25, -103.5)
- added D32: D_Small, Diode_SMD:D_0603_1608Metric_Pad1.05x0.95mm_HandSolder, F.Cu at (24.1, -104.0)
- added D33: D_Small, Diode_SMD:D_0603_1608Metric_Pad1.05x0.95mm_HandSolder, F.Cu at (49.8, -104.6)
- added D34: D_Small, Diode_SMD:D_0603_1608Metric_Pad1.05x0.95mm_HandSolder, F.Cu at (72.0, -103.6)
- added D35: D_Small, Diode_SMD:D_0603_1608Metric_Pad1.05x0.95mm_HandSolder, F.Cu at (89.0, -102.0)
- added D36: D_Small, Diode_SMD:D_0603_1608Metric_Pad1.05x0.95mm_HandSolder, F.Cu at (105.1, -103.0)
- added D37: D_Small, Diode_SMD:D_0603_1608Metric_Pad1.05x0.95mm_HandSolder, F.Cu at (126.2, -103.2)
- added D38: D_Small, Diode_SMD:D_0603_1608Metric_Pad1.05x0.95mm_HandSolder, F.Cu at (145.9, -102.8)
- added D39: D_Small, Diode_SMD:D_0603_1608Metric_Pad1.05x0.95mm_HandSolder, F.Cu at (183.4, -102.0)
- added D4: D_Small, Diode_SMD:D_0603_1608Metric_Pad1.05x0.95mm_HandSolder, F.Cu at (52.8, -158.6)
- added D40: D_Small, Diode_SMD:D_0603_1608Metric_Pad1.05x0.95mm_HandSolder, F.Cu at (166.0, -102.8)
- added D41: D_Small, Diode_SMD:D_0603_1608Metric_Pad1.05x0.95mm_HandSolder, F.Cu at (203.5, -102.2)
- added D42: D_Small, Diode_SMD:D_0603_1608Metric_Pad1.05x0.95mm_HandSolder, F.Cu at (222.5, -102.5)
- added D43: D_Small, Diode_SMD:D_0603_1608Metric_Pad1.05x0.95mm_HandSolder, F.Cu at (241.8, -102.8)
- added D44: D_Small, Diode_SMD:D_0603_1608Metric_Pad1.05x0.95mm_HandSolder, F.Cu at (261.5, -102.6)
- added D45: D_Small, Diode_SMD:D_0603_1608Metric_Pad1.05x0.95mm_HandSolder, F.Cu at (311.0, -106.2)
- added D46: MX-NoLED, Switch_Keyboard_Kailh:SW_Hotswap_Kailh_1.00u, F.Cu at (63.8, -88.8)
- added D47: D_Small, Diode_SMD:D_0603_1608Metric_Pad1.05x0.95mm_HandSolder, F.Cu at (2.50, -84.5)
- added D48: D_Small, Diode_SMD:D_0603_1608Metric_Pad1.05x0.95mm_HandSolder, F.Cu at (27.4, -84.0)
- added D49: D_Small, Diode_SMD:D_0603_1608Metric_Pad1.05x0.95mm_HandSolder, F.Cu at (50.2, -84.9)
- added D5: D_Small, Diode_SMD:D_0603_1608Metric_Pad1.05x0.95mm_HandSolder, F.Cu at (71.2, -158.2)
- added D50: D_Small, Diode_SMD:D_0603_1608Metric_Pad1.05x0.95mm_HandSolder, F.Cu at (69.5, -84.6)
- added D51: D_Small, Diode_SMD:D_0603_1608Metric_Pad1.05x0.95mm_HandSolder, F.Cu at (88.8, -83.8)
- added D52: D_Small, Diode_SMD:D_0603_1608Metric_Pad1.05x0.95mm_HandSolder, F.Cu at (108.2, -84.1)
- added D53: D_Small, Diode_SMD:D_0603_1608Metric_Pad1.05x0.95mm_HandSolder, F.Cu at (128.2, -83.4)
- added D54: D_Small, Diode_SMD:D_0603_1608Metric_Pad1.05x0.95mm_HandSolder, F.Cu at (145.5, -83.6)
- added D55: D_Small, Diode_SMD:D_0603_1608Metric_Pad1.05x0.95mm_HandSolder, F.Cu at (162.2, -82.0)
- added D56: D_Small, Diode_SMD:D_0603_1608Metric_Pad1.05x0.95mm_HandSolder, F.Cu at (183.2, -81.4)
- added D57: D_Small, Diode_SMD:D_0603_1608Metric_Pad1.05x0.95mm_HandSolder, F.Cu at (202.0, -82.0)
- added D58: D_Small, Diode_SMD:D_0603_1608Metric_Pad1.05x0.95mm_HandSolder, F.Cu at (220.5, -81.6)
- added D59: D_Small, Diode_SMD:D_0603_1608Metric_Pad1.05x0.95mm_HandSolder, F.Cu at (251.5, -80.6)
- added D6: D_Small, Diode_SMD:D_0603_1608Metric_Pad1.05x0.95mm_HandSolder, F.Cu at (93.5, -157.4)
- added D60: D_Small, Diode_SMD:D_0603_1608Metric_Pad1.05x0.95mm_HandSolder, F.Cu at (310.2, -87.1)
- added D61: D_Small, Diode_SMD:D_0603_1608Metric_Pad1.05x0.95mm_HandSolder, F.Cu at (-1.00, -62.9)
- added D62: D_Small, Diode_SMD:D_0603_1608Metric_Pad1.05x0.95mm_HandSolder, F.Cu at (30.8, -62.9)
- added D63: D_Small, Diode_SMD:D_0603_1608Metric_Pad1.05x0.95mm_HandSolder, F.Cu at (49.4, -63.2)
- added D64: D_Small, Diode_SMD:D_0603_1608Metric_Pad1.05x0.95mm_HandSolder, F.Cu at (69.8, -63.8)
- added D65: D_Small, Diode_SMD:D_0603_1608Metric_Pad1.05x0.95mm_HandSolder, F.Cu at (90.8, -63.0)
- added D66: D_Small, Diode_SMD:D_0603_1608Metric_Pad1.05x0.95mm_HandSolder, F.Cu at (117.4, -61.5)
- added D67: D_Small, Diode_SMD:D_0603_1608Metric_Pad1.05x0.95mm_HandSolder, F.Cu at (141.8, -61.8)
- added D68: D_Small, Diode_SMD:D_0603_1608Metric_Pad1.05x0.95mm_HandSolder, F.Cu at (163.5, -62.5)
- added D69: D_Small, Diode_SMD:D_0603_1608Metric_Pad1.05x0.95mm_HandSolder, F.Cu at (201.5, -61.1)
- added D7: D_Small, Diode_SMD:D_0603_1608Metric_Pad1.05x0.95mm_HandSolder, F.Cu at (116.0, -159.4)
- added D70: D_Small, Diode_SMD:D_0603_1608Metric_Pad1.05x0.95mm_HandSolder, F.Cu at (182.0, -62.1)
- added D71: D_Small, Diode_SMD:D_0603_1608Metric_Pad1.05x0.95mm_HandSolder, F.Cu at (220.2, -61.4)
- added D72: D_Small, Diode_SMD:D_0603_1608Metric_Pad1.05x0.95mm_HandSolder, F.Cu at (248.5, -61.9)
- added D73: D_Small, Diode_SMD:D_0603_1608Metric_Pad1.05x0.95mm_HandSolder, F.Cu at (287.0, -43.2)
- added D74: D_Small, Diode_SMD:D_0603_1608Metric_Pad1.05x0.95mm_HandSolder, F.Cu at (310.0, -67.5)
- added D75: D_Small, Diode_SMD:D_0603_1608Metric_Pad1.05x0.95mm_HandSolder, F.Cu at (-1.75, -39.0)
- added D76: D_Small, Diode_SMD:D_0603_1608Metric_Pad1.05x0.95mm_HandSolder, F.Cu at (22.0, -39.2)
- added D77: D_Small, Diode_SMD:D_0603_1608Metric_Pad1.05x0.95mm_HandSolder, F.Cu at (41.8, -38.9)
- added D78: D_Small, Diode_SMD:D_0603_1608Metric_Pad1.05x0.95mm_HandSolder, F.Cu at (114.5, -39.0)
- added D79: D_Small, Diode_SMD:D_0603_1608Metric_Pad1.05x0.95mm_HandSolder, F.Cu at (181.5, -42.1)
- added D8: D_Small, Diode_SMD:D_0603_1608Metric_Pad1.05x0.95mm_HandSolder, F.Cu at (133.8, -157.9)
- added D80: D_Small, Diode_SMD:D_0603_1608Metric_Pad1.05x0.95mm_HandSolder, F.Cu at (210.0, -41.0)
- added D81: D_Small, Diode_SMD:D_0603_1608Metric_Pad1.05x0.95mm_HandSolder, F.Cu at (236.0, -39.0)
- added D82: D_Small, Diode_SMD:D_0603_1608Metric_Pad1.05x0.95mm_HandSolder, F.Cu at (269.2, -24.1)
- added D83: D_Small, Diode_SMD:D_0603_1608Metric_Pad1.05x0.95mm_HandSolder, F.Cu at (288.8, -24.4)
- added D84: D_Small, Diode_SMD:D_0603_1608Metric_Pad1.05x0.95mm_HandSolder, F.Cu at (306.5, -24.0)
- added D9: D_Small, Diode_SMD:D_0603_1608Metric_Pad1.05x0.95mm_HandSolder, F.Cu at (154.0, -157.0)
- added DEL1: MX-NoLED, Switch_Keyboard_Kailh:SW_Hotswap_Kailh_1.00u, F.Cu at (261.0, -160.5)
- added DOWN1: MX-NoLED, Switch_Keyboard_Kailh:SW_Hotswap_Kailh_1.00u, F.Cu at (282.8, -29.5)
- added E1: MX-NoLED, Switch_Keyboard_Kailh:SW_Hotswap_Kailh_1.00u, F.Cu at (65.8, -108.8)
- added ENTER1: MX-NoLED, Switch_Keyboard_Kailh:SW_Hotswap_Kailh_1.00u, F.Cu at (246.0, -88.0)
- added F10: MX-NoLED, Switch_Keyboard_Kailh:SW_Hotswap_Kailh_1.00u, F.Cu at (192.8, -161.0)
- added F11: MX-NoLED, Switch_Keyboard_Kailh:SW_Hotswap_Kailh_1.00u, F.Cu at (212.8, -160.8)
- added F12: MX-NoLED, Switch_Keyboard_Kailh:SW_Hotswap_Kailh_1.00u, F.Cu at (231.8, -160.8)
- added F13: MX-NoLED, Switch_Keyboard_Kailh:SW_Hotswap_Kailh_1.00u, F.Cu at (83.2, -88.8)
- added F4: MX-NoLED, Switch_Keyboard_Kailh:SW_Hotswap_Kailh_1.00u, F.Cu at (65.0, -162.5)
- added F5: MX-NoLED, Switch_Keyboard_Kailh:SW_Hotswap_Kailh_1.00u, F.Cu at (87.2, -162.2)
- added F6: MX-NoLED, Switch_Keyboard_Kailh:SW_Hotswap_Kailh_1.00u, F.Cu at (108.0, -161.8)
- added F7: MX-NoLED, Switch_Keyboard_Kailh:SW_Hotswap_Kailh_1.00u, F.Cu at (127.8, -162.2)
- added F8: MX-NoLED, Switch_Keyboard_Kailh:SW_Hotswap_Kailh_1.00u, F.Cu at (147.5, -161.5)
- added F9: MX-NoLED, Switch_Keyboard_Kailh:SW_Hotswap_Kailh_1.00u, F.Cu at (172.5, -161.0)
- added FN1: MX-NoLED, Switch_Keyboard_Kailh:SW_Hotswap_Kailh_1.00u, F.Cu at (205.5, -46.5)
- added G1: MX-NoLED, Switch_Keyboard_Kailh:SW_Hotswap_Kailh_1.00u, F.Cu at (102.5, -89.0)
- added H1: MX-NoLED, Switch_Keyboard_Kailh:SW_Hotswap_Kailh_1.00u, F.Cu at (122.5, -88.0)
- added I1: MX-NoLED, Switch_Keyboard_Kailh:SW_Hotswap_Kailh_1.00u, F.Cu at (178.5, -107.8)
- added J1: MX-NoLED, Switch_Keyboard_Kailh:SW_Hotswap_Kailh_1.00u, F.Cu at (139.2, -88.2)
- added K1: MX-NoLED, Switch_Keyboard_Kailh:SW_Hotswap_Kailh_1.00u, F.Cu at (156.2, -88.0)
- added L1: MX-NoLED, Switch_Keyboard_Kailh:SW_Hotswap_Kailh_1.00u, F.Cu at (176.8, -87.2)
- added LEFT1: MX-NoLED, Switch_Keyboard_Kailh:SW_Hotswap_Kailh_1.00u, F.Cu at (263.8, -29.5)
- added L_SHIFT1: MX-NoLED, Switch_Keyboard_Kailh:SW_Hotswap_Kailh_1.00u, F.Cu at (-5.50, -68.2)
- added M1: MX-NoLED, Switch_Keyboard_Kailh:SW_Hotswap_Kailh_1.00u, F.Cu at (157.8, -67.0)
- added MX1: MX-NoLED, Switch_Keyboard_Kailh:SW_Hotswap_Kailh_1.00u, F.Cu at (4.75, -128.8)
- added MX10: MX-NoLED, Switch_Keyboard_Kailh:SW_Hotswap_Kailh_1.00u, F.Cu at (180.5, -129.5)
- added MX2: MX-NoLED, Switch_Keyboard_Kailh:SW_Hotswap_Kailh_1.00u, F.Cu at (24.2, -128.8)
- added MX3: MX-NoLED, Switch_Keyboard_Kailh:SW_Hotswap_Kailh_1.00u, F.Cu at (43.2, -129.0)
- added MX4: MX-NoLED, Switch_Keyboard_Kailh:SW_Hotswap_Kailh_1.00u, F.Cu at (63.5, -129.2)
- added MX5: MX-NoLED, Switch_Keyboard_Kailh:SW_Hotswap_Kailh_1.00u, F.Cu at (85.0, -129.5)
- added MX6: MX-NoLED, Switch_Keyboard_Kailh:SW_Hotswap_Kailh_1.00u, F.Cu at (104.5, -129.2)
- added MX7: MX-NoLED, Switch_Keyboard_Kailh:SW_Hotswap_Kailh_1.00u, F.Cu at (124.2, -129.2)
- added MX8: MX-NoLED, Switch_Keyboard_Kailh:SW_Hotswap_Kailh_1.00u, F.Cu at (144.0, -129.0)
- added MX9: MX-NoLED, Switch_Keyboard_Kailh:SW_Hotswap_Kailh_1.00u, F.Cu at (163.5, -129.0)
- added N1: MX-NoLED, Switch_Keyboard_Kailh:SW_Hotswap_Kailh_1.00u, F.Cu at (136.2, -67.2)
- added O1: MX-NoLED, Switch_Keyboard_Kailh:SW_Hotswap_Kailh_1.00u, F.Cu at (160.5, -107.8)
- added OPT1: MX-NoLED, Switch_Keyboard_Kailh:SW_Hotswap_Kailh_1.00u, F.Cu at (306.0, -161.5)
- added OPT2: MX-NoLED, Switch_Keyboard_Kailh:SW_Hotswap_Kailh_1.00u, F.Cu at (305.2, -130.5)
- added OPT3: MX-NoLED, Switch_Keyboard_Kailh:SW_Hotswap_Kailh_1.00u, F.Cu at (305.5, -111.2)
- added OPT4: MX-NoLED, Switch_Keyboard_Kailh:SW_Hotswap_Kailh_1.00u, F.Cu at (305.5, -92.2)
- added OPT5: MX-NoLED, Switch_Keyboard_Kailh:SW_Hotswap_Kailh_1.00u, F.Cu at (305.5, -73.0)
- added P1: MX-NoLED, Switch_Keyboard_Kailh:SW_Hotswap_Kailh_1.00u, F.Cu at (198.0, -107.5)
- added Q1: MX-NoLED, Switch_Keyboard_Kailh:SW_Hotswap_Kailh_1.00u, F.Cu at (19.5, -108.2)
- added R1: MX-NoLED, Switch_Keyboard_Kailh:SW_Hotswap_Kailh_1.00u, F.Cu at (84.0, -108.2)
- added RIGHT1: MX-NoLED, Switch_Keyboard_Kailh:SW_Hotswap_Kailh_1.00u, F.Cu at (301.8, -29.5)
- added R_SHIFT1: MX-NoLED, Switch_Keyboard_Kailh:SW_Hotswap_Kailh_1.00u, F.Cu at (243.0, -68.0)
- added S1: MX-NoLED, Switch_Keyboard_Kailh:SW_Hotswap_Kailh_1.00u, F.Cu at (44.5, -88.8)
- added SPACE1: MX-NoLED, Switch_Keyboard_Kailh:SW_Hotswap_Kailh_1.00u, F.Cu at (109.0, -44.2)
- added T1: MX-NoLED, Switch_Keyboard_Kailh:SW_Hotswap_Kailh_1.00u, F.Cu at (100.0, -107.8)
- added TAB1: MX-NoLED, Switch_Keyboard_Kailh:SW_Hotswap_Kailh_1.00u, F.Cu at (-4.75, -109.0)
- added U1: MX-NoLED, Switch_Keyboard_Kailh:SW_Hotswap_Kailh_1.00u, F.Cu at (141.0, -107.5)
- added UP1: MX-NoLED, Switch_Keyboard_Kailh:SW_Hotswap_Kailh_1.00u, F.Cu at (282.8, -48.5)
- added V1: MX-NoLED, Switch_Keyboard_Kailh:SW_Hotswap_Kailh_1.00u, F.Cu at (84.8, -68.0)
- added W1: MX-NoLED, Switch_Keyboard_Kailh:SW_Hotswap_Kailh_1.00u, F.Cu at (43.0, -108.5)
- added WIN1: MX-NoLED, Switch_Keyboard_Kailh:SW_Hotswap_Kailh_1.00u, F.Cu at (16.2, -44.0)
- added X1: MX-NoLED, Switch_Keyboard_Kailh:SW_Hotswap_Kailh_1.00u, F.Cu at (44.8, -68.0)
- added Y1: MX-NoLED, Switch_Keyboard_Kailh:SW_Hotswap_Kailh_1.00u, F.Cu at (121.0, -108.8)
- added Z1: MX-NoLED, Switch_Keyboard_Kailh:SW_Hotswap_Kailh_1.00u, F.Cu at (23.0, -67.0)
- added [1: MX-NoLED, Switch_Keyboard_Kailh:SW_Hotswap_Kailh_1.00u, F.Cu at (217.2, -107.5)
- added \1: MX-NoLED, Switch_Keyboard_Kailh:SW_Hotswap_Kailh_1.00u, F.Cu at (256.0, -107.5)
- added ]1: MX-NoLED, Switch_Keyboard_Kailh:SW_Hotswap_Kailh_1.00u, F.Cu at (236.8, -107.5)
- added `~1: MX-NoLED, Switch_Keyboard_Kailh:SW_Hotswap_Kailh_1.00u, F.Cu at (-14.0, -128.0)
- F1: renamed from MX2; footprint Switch_Keyboard_Kailh:SW_Kailh_Choc_V1_1.00u -> Switch_Keyboard_Kailh:SW_Hotswap_Kailh_1.00u
- F3: renamed from MX4; footprint Mounting_Keyboard_Stabilizer:Stabilizer_Cherry_MX_6.25u -> Switch_Keyboard_Kailh:SW_Hotswap_Kailh_1.00u
- esc1: renamed from MX1; footprint Switch_Keyboard_Kailh:SW_Hotswap_Kailh_2.25u -> Switch_Keyboard_Kailh:SW_Hotswap_Kailh_1.00u
- moved F1 273.2 mm to (7.40, -162.8)
- moved F2 262.7 mm to (26.4, -162.8)
- moved esc1 258.6 mm to (-15.6, -162.7)
- moved F3 219.1 mm to (45.5, -162.8)
- renumbered MX3 to F2
Connections:
- F1 pad 1: unconnected-(MX2-Pad1) -> Net-(A1-Pad1)
- F1 pad 2: unconnected-(MX2-Pad2) -> Net-(F1-Pad2)
- F2 pad 1: unconnected-(MX3-Pad1) -> Net-(ALT1-Pad1)
- F2 pad 2: unconnected-(MX3-Pad2) -> Net-(F2-Pad2)
- esc1 pad 1: unconnected-(MX1-Pad1) -> Net-(CAPS1-Pad1)
- esc1 pad 2: unconnected-(MX1-Pad2) -> Net-(esc1-Pad2)

Commit message: align layout
Parts:
- ALT1, CLT1, WIN1: footprint Switch_Keyboard_Kailh:SW_Hotswap_Kailh_1.00u -> Switch_Keyboard_Kailh:SW_Hotswap_Kailh_1.25u
- BACK1: footprint Switch_Keyboard_Kailh:SW_Hotswap_Kailh_1.00u -> Switch_Keyboard_Kailh:SW_Hotswap_Kailh_2.00u
- CAPS1, R_SHIFT1: footprint Switch_Keyboard_Kailh:SW_Hotswap_Kailh_1.00u -> Switch_Keyboard_Kailh:SW_Hotswap_Kailh_1.75u
- D1, D10, D11, D12, D13, D14, D15, D16, D17, D18, D19, D2, D20, D21, D22, D23, D24, D25, D26, D27, D28, D29, D3, D30, D31, D32, D33, D34, D35, D36, D37, D38, D39, D4, D40, D41, D42, D43, D44, D45, D47, D48, D49, D5, D50, D51, D52, D53, D54, D55, D56, D57, D58, D59, D6, D60, D61, D62, D63, D64, D65, D66, D67, D68, D69, D7, D70, D71, D72, D73, D74, D75, D76, D77, D78, D79, D8, D80, D81, D82, D83, D84, D9: moved to B.Cu
- ENTER1, L_SHIFT1: footprint Switch_Keyboard_Kailh:SW_Hotswap_Kailh_1.00u -> Switch_Keyboard_Kailh:SW_Hotswap_Kailh_2.25u
- SPACE1: footprint Switch_Keyboard_Kailh:SW_Hotswap_Kailh_1.00u -> Switch_Keyboard_Kailh:SW_Hotswap_Kailh_6.25u
- TAB1, \1: footprint Switch_Keyboard_Kailh:SW_Hotswap_Kailh_1.00u -> Switch_Keyboard_Kailh:SW_Hotswap_Kailh_1.50u
- moved F3 253.0 mm to (121.5, 78.6)
- moved F1 253.0 mm to (83.3, 78.6)
- moved F2 253.0 mm to (102.4, 78.6)
- moved F5 252.9 mm to (164.3, 78.6)
- moved esc1 252.7 mm to (59.5, 78.6)
- moved F4 252.6 mm to (140.5, 78.6)
- moved F7 252.2 mm to (202.4, 78.6)
- moved F6 251.9 mm to (183.4, 78.6)
- moved F8 251.2 mm to (221.5, 78.6)
- moved F9 250.4 mm to (245.3, 78.6)
- moved F10 250.0 mm to (264.3, 78.6)
- moved D7 249.7 mm to (191.8, 78.6)
- moved D3 249.6 mm to (110.9, 78.6)
- moved D2 249.6 mm to (91.8, 78.6)
- moved F12 249.5 mm to (302.4, 78.6)
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Connections:
- +1 pad 1: Net-(+1-Pad1) -> Net-(LEFT1-Pad1)
- DOWN1 pad 1: unconnected-(DOWN1-Pad1) -> Net-(BACK1-Pad1)
- ENTER1 pad 1: Net-(+1-Pad1) -> Net-(LEFT1-Pad1)
- F12 pad 1: Net-(+1-Pad1) -> Net-(LEFT1-Pad1)
- LEFT1 pad 1: unconnected-(LEFT1-Pad1) -> Net-(LEFT1-Pad1)
- UP1 pad 1: unconnected-(UP1-Pad1) -> Net-(BACK1-Pad1)
- ]1 pad 1: Net-(+1-Pad1) -> Net-(LEFT1-Pad1)

Commit message: add stabilizer hole
Parts:
- added REF**: Stabilizer_Cherry_MX_2u, Mounting_Keyboard_Stabilizer:Stabilizer_Cherry_MX_2u, F.Cu at (316.7, 107.2)
- added REF**: Stabilizer_Cherry_MX_2u, Mounting_Keyboard_Stabilizer:Stabilizer_Cherry_MX_2u, F.Cu at (314.3, 145.3)
- added REF**: Stabilizer_Cherry_MX_6.25u, Mounting_Keyboard_Stabilizer:Stabilizer_Cherry_MX_6.25u, F.Cu at (181.0, 183.4)
- added REF**: Stabilizer_Cherry_MX_2u, Mounting_Keyboard_Stabilizer:Stabilizer_Cherry_MX_2u, F.Cu at (71.4, 164.3)
- moved D14 0.85 mm to (334.7, 78.6)
Changed lines of the file:
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@@
     )
   )
+  (footprint "Mounting_Keyboard_Stabilizer:Stabilizer_Cherry_MX_2u" (layer "F.Cu")
+    (at 316.70625 107.15625)
+    (descr "Cherry MX key stabilizer 2u 2.25u 2.5u 2.75u")
+    (tags "Cherry MX key stabilizer 2u 2.25u 2.5u 2.75u")
+    (attr exclude_from_pos_files exclude_from_bom)
+    (fp_text reference "REF**" (at 0 -3) (layer "F.SilkS")
+      (effects (font (size 1 1) (thickness 0.15)))
+    )
+    (fp_text value "Stabilizer_Cherry_MX_2u" (at 0 3.2) (layer "F.Fab")
+      (effects (font (size 1 1) (thickness 0.15)))
+    )
+    (fp_text user "REF**" (at 0 0) (layer "F.Fab")
+      (effects (font (size 1 1) (thickness 0.15)))
+    )
+    (fp_line (start -2 0) (end 2 0) (layer "Dwgs.User") (width 0.1))
+    (fp_line (start 0 2) (end 0 -2) (layer "Dwgs.User") (width 0.1))
+    (pad "" np_thru_hole circle locked (at -11.938 -6.985) (size 3.048 3.048) (drill 3.048) (layers *.Cu *.Mask))
+    (pad "" np_thru_hole circle locked (at 11.938 8.255) (size 3.9878 3.9878) (drill 3.9878) (layers *.Cu *.Mask))
+    (pad "" np_thru_hole circle locked (at -11.938 8.255) (size 3.9878 3.9878) (drill 3.9878) (layers *.Cu *.Mask))
+    (pad "" np_thru_hole circle locked (at 11.938 -6.985) (size 3.048 3.048) (drill 3.048) (layers *.Cu *.Mask))
+    (model "${KICAD6_3RD_PARTY}/3dmodels/com_github_perigoso_keyswitch-kicad-library/3d-library.3dshapes/Stabilizer_Cherry_MX_2u.wrl"
+      (offset (xyz 0 0 0))
+      (scale (xyz 1 1 1))
+      (rotate (xyz 0 0 0))
+    )
+  )
   (footprint "Switch_Keyboard_Kailh:SW_Hotswap_Kailh_1.00u" (layer "F.Cu")
     (at 150.01875 145.25625)
@@
     )
   )
+  (footprint "Mounting_Keyboard_Stabilizer:Stabilizer_Cherry_MX_2u" (layer "F.Cu")
+    (at 314.325 145.25625 180)
+    (descr "Cherry MX key stabilizer 2u 2.25u 2.5u 2.75u")
+    (tags "Cherry MX key stabilizer 2u 2.25u 2.5u 2.75u")
+    (attr exclude_from_pos_files exclude_from_bom)
+    (fp_text reference "REF**" (at 0 -3) (layer "F.SilkS")
+      (effects (font (size 1 1) (thickness 0.15)))
+    )
+    (fp_text value "Stabilizer_Cherry_MX_2u" (at 0 3.2) (layer "F.Fab")
+      (effects (font (size 1 1) (thickness 0.15)))
+    )
+    (fp_text user "REF**" (at 0 0) (layer "F.Fab")
+      (effects (font (size 1 1) (thickness 0.15)))
+    )
+    (fp_line (start 0 2) (end 0 -2) (layer "Dwgs.User") (width 0.1))
+    (fp_line (start -2 0) (end 2 0) (layer "Dwgs.User") (width 0.1))
+    (pad "" np_thru_hole circle locked (at 11.938 8.255 180) (size 3.9878 3.9878) (drill 3.9878) (layers *.Cu *.Mask))
+    (pad "" np_thru_hole circle locked (at -11.938 -6.985 180) (size 3.048 3.048) (drill 3.048) (layers *.Cu *.Mask))
+    (pad "" np_thru_hole circle locked (at 11.938 -6.985 180) (size 3.048 3.048) (drill 3.048) (layers *.Cu *.Mask))
+    (pad "" np_thru_hole circle locked (at -11.938 8.255 180) (size 3.9878 3.9878) (drill 3.9878) (layers *.Cu *.Mask))
+    (model "${KICAD6_3RD_PARTY}/3dmodels/com_github_perigoso_keyswitch-kicad-library/3d-library.3dshapes/Stabilizer_Cherry_MX_2u.wrl"
+      (offset (xyz 0 0 0))
+      (scale (xyz 1 1 1))
+      (rotate (xyz 0 0 0))
+    )
+  )
   (footprint "Switch_Keyboard_Kailh:SW_Hotswap_Kailh_1.00u" (layer "F.Cu")
     (at 121.461309 78.58125)
@@
     )
   )
+  (footprint "Mounting_Keyboard_Stabilizer:Stabilizer_Cherry_MX_6.25u" (layer "F.Cu")
+    (at 180.975 183.35625 180)
+    (descr "Cherry MX key stabilizer 6.25u")
+    (tags "Cherry MX key stabilizer 6.25u")
+    (attr exclude_from_pos_files exclude_from_bom)
+    (fp_text reference "REF**" (at 0 -3) (layer "F.SilkS")
+      (effects (font (size 1 1) (thickness 0.15)))
+    )
+    (fp_text value "Stabilizer_Cherry_MX_6.25u" (at 0 3.2) (layer "F.Fab")
+      (effects (font (size 1 1) (thickness 0.15)))
+    )
+    (fp_text user "REF**" (at 0 0) (layer "F.Fab")
+      (effects (font (size 1 1) (thickness 0.15)))
+    )
+    (fp_line (start 0 2) (end 0 -2) (layer "Dwgs.User") (width 0.1))
+    (fp_line (start -2 0) (end 2 0) (layer "Dwgs.User") (width 0.1))
+    (pad "" np_thru_hole circle locked (at -50 8.255 180) (size 3.9878 3.9878) (drill 3.9878) (layers *.Cu *.Mask))
+    (pad "" np_thru_hole circle locked (at 50 -6.985 180) (size 3.048 3.048) (drill 3.048) (layers *.Cu *.Mask))
+    (pad "" np_thru_hole circle locked (at -50 -6.985 180) (size 3.048 3.048) (drill 3.048) (layers *.Cu *.Mask))
+    (pad "" np_thru_hole circle locked (at 50 8.255 180) (size 3.9878 3.9878) (drill 3.9878) (layers *.Cu *.Mask))
+    (model "${KICAD6_3RD_PARTY}/3dmodels/com_github_perigoso_keyswitch-kicad-library/3d-library.3dshapes/Stabilizer_Cherry_MX_6_25u.wrl"
+      (offset (xyz 0 0 0))
+      (scale (xyz 1 1 1))
+      (rotate (xyz 0 0 0))
+    )
+  )
   (footprint "Switch_Keyboard_Kailh:SW_Hotswap_Kailh_1.00u" (layer "F.Cu")
     (at 221.520534 78.58125)
@@
     )
   )
+  (footprint "Mounting_Keyboard_Stabilizer:Stabilizer_Cherry_MX_2u" (layer "F.Cu")
+    (at 71.4375 164.30625)
+    (descr "Cherry MX key stabilizer 2u 2.25u 2.5u 2.75u")
+    (tags "Cherry MX key stabilizer 2u 2.25u 2.5u 2.75u")
+    (attr exclude_from_pos_files exclude_from_bom)
+    (fp_text reference "REF**" (at 0 -3) (layer "F.SilkS")
+      (effects (font (size 1 1) (thickness 0.15)))
+    )
+    (fp_text value "Stabilizer_Cherry_MX_2u" (at 0 3.2) (layer "F.Fab")
+      (effects (font (size 1 1) (thickness 0.15)))
+    )
+    (fp_text user "REF**" (at 0 0) (layer "F.Fab")
+      (effects (font (size 1 1) (thickness 0.15)))
+    )
+    (fp_line (start -2 0) (end 2 0) (layer "Dwgs.User") (width 0.1))
+    (fp_line (start 0 2) (end 0 -2) (layer "Dwgs.User") (width 0.1))
+    (pad "" np_thru_hole circle locked (at 11.938 -6.985) (size 3.048 3.048) (drill 3.048) (layers *.Cu *.Mask))
+    (pad "" np_thru_hole circle locked (at -11.938 -6.985) (size 3.048 3.048) (drill 3.048) (layers *.Cu *.Mask))
+    (pad "" np_thru_hole circle locked (at 11.938 8.255) (size 3.9878 3.9878) (drill 3.9878) (layers *.Cu *.Mask))
+    (pad "" np_thru_hole circle locked (at -11.938 8.255) (size 3.9878 3.9878) (drill 3.9878) (layers *.Cu *.Mask))
+    (model "${KICAD6_3RD_PARTY}/3dmodels/com_github_perigoso_keyswitch-kicad-library/3d-library.3dshapes/Stabilizer_Cherry_MX_2u.wrl"
+      (offset (xyz 0 0 0))
+      (scale (xyz 1 1 1))
+      (rotate (xyz 0 0 0))
+    )
+  )
   (footprint "Switch_Keyboard_Kailh:SW_Hotswap_Kailh_1.00u" (layer "F.Cu")
     (at 59.53125 78.58125)
@@
   )
   (footprint "Diode_SMD:D_0603_1608Metric_Pad1.05x0.95mm_HandSolder" (layer "B.Cu")
-    (at 333.85125 78.55875 90)
+    (at 334.7 78.575 90)
     (descr "Diode SMD 0603 (1608 Metric), square (rectangular) end terminal, IPC_7351 nominal, (Body size source: http://www.tortai-tech.com/upload/download/2011102023233369053.pdf), generated with kicad-footprint-generator")
     (tags "diode handsolder")

Commit message: routing pcb
Parts:
- removed REF** (x3): Stabilizer_Cherry_MX_2u, Mounting_Keyboard_Stabilizer:Stabilizer_Cherry_MX_2u
- removed REF**: Stabilizer_Cherry_MX_6.25u, Mounting_Keyboard_Stabilizer:Stabilizer_Cherry_MX_6.25u
- added C2: 22pF, Capacitor_SMD:C_0603_1608Metric, B.Cu at (202.2, 183.4)
- added C3: 22pF, Capacitor_SMD:C_0603_1608Metric, B.Cu at (202.2, 190.6)
- added C4: 0.1uF, Capacitor_SMD:C_0603_1608Metric, B.Cu at (216.0, 196.0)
- added C5: 0.1uF, Capacitor_SMD:C_0603_1608Metric, B.Cu at (233.0, 190.2)
- added C6: 0.1uF, Capacitor_SMD:C_0603_1608Metric, B.Cu at (230.6, 190.2)
- added C7: 0.1uF, Capacitor_SMD:C_0603_1608Metric, B.Cu at (228.2, 190.2)
- added C8: 100uF, Capacitor_SMD:C_0603_1608Metric, B.Cu at (226.0, 190.2)
- added R2: 10k, Resistor_SMD:R_0603_1608Metric, B.Cu at (210.2, 193.0)
- added R3: 22, Resistor_SMD:R_0603_1608Metric, B.Cu at (227.0, 197.0)
- added R4: 22, Resistor_SMD:R_0603_1608Metric, B.Cu at (227.0, 195.0)
- added R5: 10k, Resistor_SMD:R_0603_1608Metric, B.Cu at (225.8, 178.0)
- added SW1: RotaryEncoder_Switch, Rotary_Encoder:RotaryEncoder_Alps_EC11E-Switch_Vertical_H20mm, B.Cu at (357.3, 86.1)
- added U2: ATmega32U4-A, Package_QFP:TQFP-44_10x10mm_P0.8mm, B.Cu at (217.0, 185.0)
- added Y2: Crystal_GND24_Small, Crystal:Crystal_SMD_3225-4Pin_3.2x2.5mm, B.Cu at (202.2, 187.1)
- D1, D10, D11, D12, D13, D14, D15, D16, D17, D18, D19, D2, D20, D21, D22, D23, D24, D25, D26, D27, D28, D29, D3, D30, D31, D32, D33, D34, D35, D36, D37, D38, D39, D4, D40, D41, D42, D43, D44, D45, D47, D48, D49, D5, D50, D51, D52, D53, D54, D55, D56, D57, D58, D59, D6, D60, D61, D62, D63, D64, D65, D66, D67, D68, D69, D7, D70, D71, D72, D73, D74, D75, D76, D77, D78, D79, D8, D80, D81, D82, D83, D84, D9: footprint Diode_SMD:D_0603_1608Metric_Pad1.05x0.95mm_HandSolder -> Diode_SMD:D_SOD-123
Connections:
- net Net-('1-Pad1) renamed COL12
- net Net-(,1-Pad1) renamed COL9
- net Net-(.1-Pad1) renamed COL10
- net Net-(/1-Pad1) renamed COL11
- net Net-(A1-Pad1) renamed COL2
- net Net-(ALT1-Pad1) renamed COL3
- net Net-(B1-Pad1) renamed COL6
- net Net-(BACK1-Pad1) renamed COL14
- net Net-(C1-Pad1) renamed COL4
- net Net-(CAPS1-Pad1) renamed COL1
- net Net-(D1-Pad1) renamed ROW1
- net Net-(D16-Pad1) renamed ROW2
- net Net-(D31-Pad1) renamed ROW3
- net Net-(D47-Pad1) renamed ROW4
- net Net-(D61-Pad1) renamed ROW5
- net Net-(D75-Pad1) renamed ROW6
- net Net-(F13-Pad1) renamed COL5
- net Net-(F6-Pad1) renamed COL7
- net Net-(F7-Pad1) renamed COL8
- net Net-(LEFT1-Pad1) renamed COL13
- net Net-(OPT1-Pad1) renamed COL15
- net Net-(OPT1-Pad2) renamed /ROT1
Routing:
- net ROW2: track 0.00 -> 447.8 mm, vias 0 -> 6
- net ROW3: track 0.00 -> 415.6 mm, vias 0 -> 4
- net ROW4: track 0.00 -> 390.2 mm, vias 0 -> 2
- net ROW6: track 0.00 -> 348.8 mm, vias 0 -> 2
- net ROW5: track 0.00 -> 308.3 mm
- net ROW1: track 0.00 -> 304.0 mm
- net COL15: track 0.00 -> 293.5 mm, vias 0 -> 6
- net GND: track 0.00 -> 292.7 mm, vias 0 -> 6
- net COL1: track 0.00 -> 276.0 mm, vias 0 -> 2
- net ROT_A: track 0.00 -> 269.9 mm, vias 0 -> 1
- net ROT_B: track 0.00 -> 264.6 mm, vias 0 -> 1
- net COL2: track 0.00 -> 261.1 mm, vias 0 -> 11
- net COL14: track 0.00 -> 243.7 mm, vias 0 -> 6
- net COL3: track 0.00 -> 243.4 mm, vias 0 -> 6
- net COL13: track 0.00 -> 232.7 mm, vias 0 -> 6
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Other:
- board outline added: 319.1 x 133.4 mm

Commit message: fix some missing footprint
Parts:
- added REF**: Stabilizer_Cherry_MX_2u, Mounting_Keyboard_Stabilizer:Stabilizer_Cherry_MX_2u, F.Cu at (330.6, 143.7)
- added REF**: Stabilizer_Cherry_MX_6.25u, Mounting_Keyboard_Stabilizer:Stabilizer_Cherry_MX_6.25u, F.Cu at (197.2, 181.8)
- added REF**: TestPoint_THTPad_D1.0mm_Drill0.5mm, TestPoint:TestPoint_THTPad_D1.0mm_Drill0.5mm, F.Cu at (223.6, 194.8)
- added REF**: Stabilizer_Cherry_MX_2u, Mounting_Keyboard_Stabilizer:Stabilizer_Cherry_MX_2u, F.Cu at (333.0, 105.6)
- added REF**: Stabilizer_Cherry_MX_2u, Mounting_Keyboard_Stabilizer:Stabilizer_Cherry_MX_2u, F.Cu at (87.7, 162.8)
- added REF**: TestPoint_THTPad_1.0x1.0mm_Drill0.5mm, TestPoint:TestPoint_THTPad_1.0x1.0mm_Drill0.5mm, F.Cu at (223.6, 192.4)
- moved C5 24.0 mm to (256.8, 193.7)
- moved C6 24.0 mm to (254.3, 193.7)
- moved C7 24.0 mm to (252.0, 193.7)
- moved C8 24.0 mm to (249.8, 193.7)
- moved DOWN1 16.3 mm to (347.3, 186.6)
- moved '1 16.3 mm to (299.6, 143.7)
- moved D41 16.3 mm to (284.2, 124.6)
- moved D57 16.3 mm to (289.0, 143.7)
- moved D84 16.3 mm to (374.8, 186.5)
- moved OPT1 16.3 mm to (371.1, 77.0)
- moved OPT2 16.3 mm to (371.1, 105.6)
- moved OPT3 16.3 mm to (371.1, 124.7)
- moved OPT4 16.3 mm to (371.1, 143.7)
- moved OPT5 16.3 mm to (371.1, 162.8)
- moved P1 16.3 mm to (275.8, 124.7)
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Routing:
- net +5V: track 35.3 -> 64.2 mm
- net GND: track 292.7 -> 308.6 mm, vias 6 -> 7
- net COL12: track 196.6 -> 209.0 mm, vias 3 -> 7
- net COL9: track 126.8 -> 134.9 mm, vias 3 -> 6
- net COL7: track 135.6 -> 142.3 mm, vias 3 -> 6
- net COL14: track 243.7 -> 237.6 mm
- net Net-(D5-Pad2): track 0.00 -> 4.51 mm
- net COL5: track 180.4 -> 184.6 mm
- net COL3: track 243.4 -> 246.5 mm, vias 6 -> 7
- net Net-(R4-Pad2): track 9.08 -> 9.89 mm
Other:
- board size 319.1 x 133.4 mm -> 319.1 x 133.3 mm

Commit message: add type c and expand power
Parts:
- added F14: 500mA, Fuse:Fuse_1206_3216Metric, B.Cu at (222.5, 160.4)
- added J2: USB_C_Receptacle_USB2.0, Connector_USB:USB_C_Receptacle_GCT_USB4085, F.Cu at (326.4, 54.5)
- moved C5 50.0 mm to (218.4, 161.7)
- moved C6 50.0 mm to (216.0, 161.7)
- moved C7 50.0 mm to (213.6, 161.7)
- moved C8 50.0 mm to (211.4, 161.7)
- moved OPT4 37.3 mm to (337.7, 127.1)
- moved OPT5 37.3 mm to (337.7, 146.1)
- moved UP1 37.3 mm to (313.9, 150.9)
- moved '1 37.3 mm to (266.3, 127.0)
- moved +1 37.3 mm to (271.1, 88.9)
- moved D29 37.3 mm to (307.9, 88.9)
- moved D41 37.3 mm to (250.9, 108.0)
- moved D42 37.3 mm to (269.9, 108.0)
- moved D44 37.3 mm to (312.6, 108.0)
- moved D57 37.3 mm to (255.7, 127.0)
- moved OPT2 37.3 mm to (337.7, 88.9)
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Routing:
- net D+: track 0.00 -> 237.5 mm, vias 0 -> 1
- net D-: track 0.17 -> 236.9 mm, vias 0 -> 1
- net VCC: track 0.00 -> 209.1 mm, vias 0 -> 1
- net GND: track 308.6 -> 320.1 mm, vias 7 -> 9
- net +5V: track 64.2 -> 73.4 mm

Commit message: fix2
Parts:
- removed the REF** at (190.2, 178.1)
- removed the REF** at (190.2, 175.8)
- added TP1: RESET, TestPoint:TestPoint_THTPad_1.0x1.0mm_Drill0.5mm, F.Cu at (194.6, 176.3)
- added TP2: GND, TestPoint:TestPoint_THTPad_D1.0mm_Drill0.5mm, F.Cu at (194.6, 178.4)
Routing:
- net ROT_A: track 269.9 -> 256.5 mm
- net GND: track 320.1 -> 326.8 mm
- net ROT_B: track 264.6 -> 257.9 mm
- net ROW6: track 348.8 -> 343.0 mm
- net Net-(R2-Pad2): track 6.34 -> 8.13 mm
