File: fese75.kicad_pcb (KiCad board)
At the start: 2 copper layers, 319.1 x 133.3 mm, 188 parts, among them J1 MX-NoLED, J2 USB_C_Receptacle_USB2.0, K1 MX-NoLED, M1 MX-NoLED, P1 MX-NoLED, Q1 MX-NoLED, SW1 RotaryEncoder_Switch, T1 MX-NoLED, U1 MX-NoLED, U2 ATmega32U4-A, X1 MX-NoLED, Y1 MX-NoLED, Y2 Crystal_GND24_Small

Commit message: add testpoint
Parts:
- added TP10: TestPoint, TestPoint:TestPoint_THTPad_D2.0mm_Drill1.0mm, F.Cu at (178.5, 76.0)
- added TP11: TestPoint, TestPoint:TestPoint_THTPad_D2.0mm_Drill1.0mm, F.Cu at (182.4, 76.0)
- added TP12: TestPoint, TestPoint:TestPoint_THTPad_D2.0mm_Drill1.0mm, F.Cu at (186.3, 76.0)
- added TP13: TestPoint, TestPoint:TestPoint_THTPad_D2.0mm_Drill1.0mm, F.Cu at (190.1, 76.0)
- added TP14: TestPoint, TestPoint:TestPoint_THTPad_D2.0mm_Drill1.0mm, F.Cu at (194.0, 76.0)
- added TP15: TestPoint, TestPoint:TestPoint_THTPad_D2.0mm_Drill1.0mm, F.Cu at (197.9, 76.0)
- added TP16: TestPoint, TestPoint:TestPoint_THTPad_D2.0mm_Drill1.0mm, F.Cu at (201.8, 76.0)
- added TP17: TestPoint, TestPoint:TestPoint_THTPad_D2.0mm_Drill1.0mm, F.Cu at (205.6, 76.0)
- added TP18: TestPoint, TestPoint:TestPoint_THTPad_2.0x2.0mm_Drill1.0mm, F.Cu at (232.5, 154.3)
- added TP19: TestPoint, TestPoint:TestPoint_THTPad_D2.0mm_Drill1.0mm, F.Cu at (236.4, 154.3)
- added TP20: TestPoint, TestPoint:TestPoint_THTPad_D2.0mm_Drill1.0mm, F.Cu at (240.2, 154.3)
- added TP21: TestPoint, TestPoint:TestPoint_THTPad_D2.0mm_Drill1.0mm, F.Cu at (244.0, 154.3)
- added TP22: TestPoint, TestPoint:TestPoint_THTPad_D2.0mm_Drill1.0mm, F.Cu at (247.8, 154.3)
- added TP23: TestPoint, TestPoint:TestPoint_THTPad_D2.0mm_Drill1.0mm, F.Cu at (251.6, 154.3)
- added TP3: CO1, TestPoint:TestPoint_THTPad_2.0x2.0mm_Drill1.0mm, F.Cu at (151.3, 75.9)
- added TP4: CO2, TestPoint:TestPoint_THTPad_D2.0mm_Drill1.0mm, F.Cu at (155.2, 75.9)
- added TP5: CO3, TestPoint:TestPoint_THTPad_D2.0mm_Drill1.0mm, F.Cu at (159.1, 75.9)
- added TP6: CO4, TestPoint:TestPoint_THTPad_D2.0mm_Drill1.0mm, F.Cu at (163.0, 75.9)
- added TP7: TestPoint, TestPoint:TestPoint_THTPad_D2.0mm_Drill1.0mm, F.Cu at (166.9, 76.0)
- added TP8: TestPoint, TestPoint:TestPoint_THTPad_D2.0mm_Drill1.0mm, F.Cu at (170.7, 76.0)
- added TP9: TestPoint, TestPoint:TestPoint_THTPad_D2.0mm_Drill1.0mm, F.Cu at (174.6, 76.0)
- TP1: footprint TestPoint:TestPoint_THTPad_1.0x1.0mm_Drill0.5mm -> TestPoint:TestPoint_THTPad_2.0x2.0mm_Drill1.0mm
- TP2: footprint TestPoint:TestPoint_THTPad_D1.0mm_Drill0.5mm -> TestPoint:TestPoint_THTPad_D2.0mm_Drill1.0mm
Connections:
- U2 pad 11: unconnected-(U2-Pad11) -> ROW1
Routing:
- net ROW1: track 304.0 -> 666.2 mm, vias 0 -> 6
- net COL1: track 276.0 -> 406.9 mm, vias 2 -> 6
- net COL15: track 293.5 -> 422.8 mm, vias 6 -> 7
- net COL13: track 232.7 -> 356.5 mm
- net COL4: track 203.1 -> 320.1 mm
- net COL2: track 261.1 -> 367.8 mm
- net COL12: track 209.0 -> 303.2 mm
- net COL14: track 237.6 -> 331.3 mm
- net COL5: track 184.6 -> 271.8 mm
- net COL3: track 246.5 -> 316.0 mm
- net COL11: track 176.6 -> 240.0 mm
- net COL6: track 178.3 -> 228.9 mm
- net COL10: track 157.2 -> 189.2 mm
- net COL7: track 142.3 -> 163.4 mm
- net ROW6: track 343.0 -> 361.2 mm, vias 2 -> 3
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