File: fese75.kicad_sch (KiCad schematic)
At the start: 166 parts

Commit message: quick place component
Parts:
- '1: renamed from '; footprint Switch_Keyboard_Kailh:SW_Kailh_Choc_V1_1.00u -> Switch_Keyboard_Kailh:SW_Hotswap_Kailh_1.00u
- ,1: renamed from ,; footprint Mounting_Keyboard_Stabilizer:Stabilizer_Cherry_MX_6.25u -> Switch_Keyboard_Kailh:SW_Hotswap_Kailh_1.00u
- -1: renamed from -; footprint Switch_Keyboard_Kailh:SW_Kailh_Choc_V1_1.00u -> Switch_Keyboard_Kailh:SW_Hotswap_Kailh_1.00u
- .1: renamed from .; footprint Switch_Keyboard_Kailh:SW_Hotswap_Kailh_2.25u -> Switch_Keyboard_Kailh:SW_Hotswap_Kailh_1.00u
- /1: renamed from /; footprint Switch_Keyboard_Kailh:SW_Hotswap_Kailh_2.25u -> Switch_Keyboard_Kailh:SW_Hotswap_Kailh_1.00u
- ;1: renamed from ;; footprint Switch_Keyboard_Kailh:SW_Hotswap_Kailh_2.25u -> Switch_Keyboard_Kailh:SW_Hotswap_Kailh_1.00u
- A1: renamed from A; footprint Switch_Keyboard_Kailh:SW_Kailh_Choc_V1_1.00u -> Switch_Keyboard_Kailh:SW_Hotswap_Kailh_1.00u
- ALT2: renamed from ALT; footprint Switch_Keyboard_Kailh:SW_Hotswap_Kailh_2.25u -> Switch_Keyboard_Kailh:SW_Hotswap_Kailh_1.00u
- B1: renamed from B; footprint Switch_Keyboard_Kailh:SW_Hotswap_Kailh_2.25u -> Switch_Keyboard_Kailh:SW_Hotswap_Kailh_1.00u
- BACK1: renamed from BACK; footprint Mounting_Keyboard_Stabilizer:Stabilizer_Cherry_MX_6.25u -> Switch_Keyboard_Kailh:SW_Hotswap_Kailh_1.00u
- C1: renamed from C; footprint Mounting_Keyboard_Stabilizer:Stabilizer_Cherry_MX_6.25u -> Switch_Keyboard_Kailh:SW_Hotswap_Kailh_1.00u
- CAPS1: renamed from CAPS; footprint Switch_Keyboard_Kailh:SW_Hotswap_Kailh_2.25u -> Switch_Keyboard_Kailh:SW_Hotswap_Kailh_1.00u
- CLT1: renamed from CLT; footprint Switch_Keyboard_Kailh:SW_Hotswap_Kailh_2.25u -> Switch_Keyboard_Kailh:SW_Hotswap_Kailh_1.00u
- CTL1: renamed from CTL; footprint Switch_Keyboard_Kailh:SW_Kailh_Choc_V1_1.00u -> Switch_Keyboard_Kailh:SW_Hotswap_Kailh_1.00u
- D1, D10, D11, D12, D13, D14, D15, D16, D17, D18, D19, D2, D20, D21, D22, D23, D24, D25, D26, D27, D28, D29, D3, D30, D31, D32, D33, D34, D35, D36, D37, D38, D39, D4, D40, D41, D42, D43, D44, D45, D47, D48, D49, D5, D50, D51, D52, D53, D54, D55, D56, D57, D58, D59, D6, D60, D61, D62, D63, D64, D65, D66, D67, D68, D69, D7, D70, D71, D72, D73, D74, D75, D76, D77, D78, D79, D8, D80, D81, D82, D83, D84, D9: renamed from D?; footprint (none) -> Diode_SMD:D_0603_1608Metric_Pad1.05x0.95mm_HandSolder
- D46: renamed from D; footprint Mounting_Keyboard_Stabilizer:Stabilizer_Cherry_MX_6.25u -> Switch_Keyboard_Kailh:SW_Hotswap_Kailh_1.00u
- DEL1: renamed from DEL; footprint Mounting_Keyboard_Stabilizer:Stabilizer_Cherry_MX_6.25u -> Switch_Keyboard_Kailh:SW_Hotswap_Kailh_1.00u
- DOWN1: renamed from DOWN; footprint Mounting_Keyboard_Stabilizer:Stabilizer_Cherry_MX_6.25u -> Switch_Keyboard_Kailh:SW_Hotswap_Kailh_1.00u
- E1: renamed from E; footprint Mounting_Keyboard_Stabilizer:Stabilizer_Cherry_MX_6.25u -> Switch_Keyboard_Kailh:SW_Hotswap_Kailh_1.00u
- F1, F11, F6, MX1, MX6: footprint Switch_Keyboard_Kailh:SW_Kailh_Choc_V1_1.00u -> Switch_Keyboard_Kailh:SW_Hotswap_Kailh_1.00u
- F10, F4, F5, F9, MX10, MX4, MX5, MX9, OPT2, OPT3, OPT4, OPT5: footprint Switch_Keyboard_Kailh:SW_Hotswap_Kailh_2.25u -> Switch_Keyboard_Kailh:SW_Hotswap_Kailh_1.00u
- F13: renamed from F; footprint Switch_Keyboard_Kailh:SW_Hotswap_Kailh_2.25u -> Switch_Keyboard_Kailh:SW_Hotswap_Kailh_1.00u
- F3, F8, MX3, MX8: footprint Mounting_Keyboard_Stabilizer:Stabilizer_Cherry_MX_6.25u -> Switch_Keyboard_Kailh:SW_Hotswap_Kailh_1.00u
- FN1: renamed from FN; footprint Switch_Keyboard_Kailh:SW_Hotswap_Kailh_2.25u -> Switch_Keyboard_Kailh:SW_Hotswap_Kailh_1.00u
- G1: renamed from G; footprint Switch_Keyboard_Kailh:SW_Hotswap_Kailh_2.25u -> Switch_Keyboard_Kailh:SW_Hotswap_Kailh_1.00u
- H1: renamed from H; footprint Switch_Keyboard_Kailh:SW_Kailh_Choc_V1_1.00u -> Switch_Keyboard_Kailh:SW_Hotswap_Kailh_1.00u
- I1: renamed from I; footprint Mounting_Keyboard_Stabilizer:Stabilizer_Cherry_MX_6.25u -> Switch_Keyboard_Kailh:SW_Hotswap_Kailh_1.00u
- K1: renamed from K; footprint Mounting_Keyboard_Stabilizer:Stabilizer_Cherry_MX_6.25u -> Switch_Keyboard_Kailh:SW_Hotswap_Kailh_1.00u
- L1: renamed from L; footprint Switch_Keyboard_Kailh:SW_Hotswap_Kailh_2.25u -> Switch_Keyboard_Kailh:SW_Hotswap_Kailh_1.00u
- L_SHIFT1: renamed from L_SHIFT; footprint Switch_Keyboard_Kailh:SW_Hotswap_Kailh_2.25u -> Switch_Keyboard_Kailh:SW_Hotswap_Kailh_1.00u
- N1: renamed from N; footprint Switch_Keyboard_Kailh:SW_Kailh_Choc_V1_1.00u -> Switch_Keyboard_Kailh:SW_Hotswap_Kailh_1.00u
- O1: renamed from O; footprint Switch_Keyboard_Kailh:SW_Hotswap_Kailh_2.25u -> Switch_Keyboard_Kailh:SW_Hotswap_Kailh_1.00u
- OPT1: renamed from OPT; footprint Switch_Keyboard_Kailh:SW_Hotswap_Kailh_2.25u -> Switch_Keyboard_Kailh:SW_Hotswap_Kailh_1.00u
- P1: renamed from P; footprint Switch_Keyboard_Kailh:SW_Hotswap_Kailh_2.25u -> Switch_Keyboard_Kailh:SW_Hotswap_Kailh_1.00u
- Q1: renamed from Q; footprint Switch_Keyboard_Kailh:SW_Kailh_Choc_V1_1.00u -> Switch_Keyboard_Kailh:SW_Hotswap_Kailh_1.00u
- R1: renamed from R; footprint Switch_Keyboard_Kailh:SW_Hotswap_Kailh_2.25u -> Switch_Keyboard_Kailh:SW_Hotswap_Kailh_1.00u
- RIGHT1: renamed from RIGHT; footprint Switch_Keyboard_Kailh:SW_Hotswap_Kailh_2.25u -> Switch_Keyboard_Kailh:SW_Hotswap_Kailh_1.00u
- R_SHIFT1: renamed from R_SHIFT; footprint Switch_Keyboard_Kailh:SW_Kailh_Choc_V1_1.00u -> Switch_Keyboard_Kailh:SW_Hotswap_Kailh_1.00u
- SPACE1: renamed from SPACE; footprint Switch_Keyboard_Kailh:SW_Kailh_Choc_V1_1.00u -> Switch_Keyboard_Kailh:SW_Hotswap_Kailh_1.00u
- T1: renamed from T; footprint Switch_Keyboard_Kailh:SW_Hotswap_Kailh_2.25u -> Switch_Keyboard_Kailh:SW_Hotswap_Kailh_1.00u
- TAB1: renamed from TAB; footprint Switch_Keyboard_Kailh:SW_Hotswap_Kailh_2.25u -> Switch_Keyboard_Kailh:SW_Hotswap_Kailh_1.00u
- UP1: renamed from UP; footprint Mounting_Keyboard_Stabilizer:Stabilizer_Cherry_MX_6.25u -> Switch_Keyboard_Kailh:SW_Hotswap_Kailh_1.00u
- V1: renamed from V; footprint Switch_Keyboard_Kailh:SW_Hotswap_Kailh_2.25u -> Switch_Keyboard_Kailh:SW_Hotswap_Kailh_1.00u
- WIN1: renamed from WIN; footprint Switch_Keyboard_Kailh:SW_Kailh_Choc_V1_1.00u -> Switch_Keyboard_Kailh:SW_Hotswap_Kailh_1.00u
- Y1: renamed from Y; footprint Switch_Keyboard_Kailh:SW_Kailh_Choc_V1_1.00u -> Switch_Keyboard_Kailh:SW_Hotswap_Kailh_1.00u
- Z1: renamed from Z; footprint Switch_Keyboard_Kailh:SW_Kailh_Choc_V1_1.00u -> Switch_Keyboard_Kailh:SW_Hotswap_Kailh_1.00u
- [1: renamed from [; footprint Switch_Keyboard_Kailh:SW_Kailh_Choc_V1_1.00u -> Switch_Keyboard_Kailh:SW_Hotswap_Kailh_1.00u
- \1: renamed from \; footprint Mounting_Keyboard_Stabilizer:Stabilizer_Cherry_MX_6.25u -> Switch_Keyboard_Kailh:SW_Hotswap_Kailh_1.00u
- `~1: renamed from `~; footprint Switch_Keyboard_Kailh:SW_Hotswap_Kailh_2.25u -> Switch_Keyboard_Kailh:SW_Hotswap_Kailh_1.00u
- esc1: renamed from esc; footprint Switch_Keyboard_Kailh:SW_Hotswap_Kailh_2.25u -> Switch_Keyboard_Kailh:SW_Hotswap_Kailh_1.00u
- renumbered + to +1, ALT to ALT1, ENTER to ENTER1, J to J1, LEFT to LEFT1, M to M1, S to S1, U to U1, W to W1, X to X1, ] to ]1

Commit message: align layout
Parts:
- ALT1, CLT1, WIN1: footprint Switch_Keyboard_Kailh:SW_Hotswap_Kailh_1.00u -> Switch_Keyboard_Kailh:SW_Hotswap_Kailh_1.25u
- BACK1: footprint Switch_Keyboard_Kailh:SW_Hotswap_Kailh_1.00u -> Switch_Keyboard_Kailh:SW_Hotswap_Kailh_2.00u
- CAPS1, R_SHIFT1: footprint Switch_Keyboard_Kailh:SW_Hotswap_Kailh_1.00u -> Switch_Keyboard_Kailh:SW_Hotswap_Kailh_1.75u
- ENTER1, L_SHIFT1: footprint Switch_Keyboard_Kailh:SW_Hotswap_Kailh_1.00u -> Switch_Keyboard_Kailh:SW_Hotswap_Kailh_2.25u
- SPACE1: footprint Switch_Keyboard_Kailh:SW_Hotswap_Kailh_1.00u -> Switch_Keyboard_Kailh:SW_Hotswap_Kailh_6.25u
- TAB1, \1: footprint Switch_Keyboard_Kailh:SW_Hotswap_Kailh_1.00u -> Switch_Keyboard_Kailh:SW_Hotswap_Kailh_1.50u
Connections:
- net at +1.1 (COL), ENTER1.1 (COL), F12.1 (COL)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: now also LEFT1.1 (COL)
- net at UP1.1 (COL): now also BACK1.1 (COL), DEL1.1 (COL), DOWN1.1 (COL), \1.1 (COL)
Changed lines of the file:
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@@
   (junction (at 204.47 118.11) (diameter 0) (color 0 0 0 0)
   )
+  (junction (at 232.41 107.95) (diameter 0) (color 0 0 0 0)
+  )
   (junction (at 182.88 58.42) (diameter 0) (color 0 0 0 0)
   )
@@
   (junction (at 203.2 91.44) (diameter 0) (color 0 0 0 0)
   )
+  (junction (at 242.57 124.46) (diameter 0) (color 0 0 0 0)
+  )
   (junction (at 134.62 118.11) (diameter 0) (color 0 0 0 0)
   )
@@
   (junction (at 234.95 68.58) (diameter 0) (color 0 0 0 0)
   )
+  (junction (at 242.57 91.44) (diameter 0) (color 0 0 0 0)
+  )
   (junction (at 193.04 74.93) (diameter 0) (color 0 0 0 0)
   )
@@
     (stroke (width 0) (type default) (color 0 0 0 0))
   )
+  (wire (pts (xy 232.41 107.95) (xy 232.41 140.97))
+    (stroke (width 0) (type default) (color 0 0 0 0))
+  )
   (wire (pts (xy 154.94 63.5) (xy 157.48 63.5))
     (stroke (width 0) (type default) (color 0 0 0 0))
@@
     (stroke (width 0) (type default) (color 0 0 0 0))
   )
+  (wire (pts (xy 242.57 124.46) (xy 242.57 140.97))
+    (stroke (width 0) (type default) (color 0 0 0 0))
+  )
   (wire (pts (xy 111.76 91.44) (xy 111.76 107.95))
     (stroke (width 0) (type default) (color 0 0 0 0))
@@
     (stroke (width 0) (type default) (color 0 0 0 0))
   )
+  (wire (pts (xy 242.57 91.44) (xy 242.57 124.46))
+    (stroke (width 0) (type default) (color 0 0 0 0))
+  )
   (wire (pts (xy 203.2 50.8) (xy 203.2 58.42))
     (stroke (width 0) (type default) (color 0 0 0 0))
@@
       (effects (font (size 0.508 0.508)))
     )
-    (property "Footprint" "Switch_Keyboard_Kailh:SW_Hotswap_Kailh_1.00u" (id 2) (at 92.075 93.345 0)
+    (property "Footprint" "Switch_Keyboard_Kailh:SW_Hotswap_Kailh_1.50u" (id 2) (at 92.075 93.345 0)
       (effects (font (size 1.524 1.524)) hide)
     )
@@
       (effects (font (size 0.508 0.508)))
     )
-    (property "Footprint" "Switch_Keyboard_Kailh:SW_Hotswap_Kailh_1.00u" (id 2) (at 92.075 109.855 0)
+    (property "Footprint" "Switch_Keyboard_Kailh:SW_Hotswap_Kailh_1.75u" (id 2) (at 92.075 109.855 0)
       (effects (font (size 1.524 1.524)) hide)
     )
@@
       (effects (font (size 0.508 0.508)))
     )
-    (property "Footprint" "Switch_Keyboard_Kailh:SW_Hotswap_Kailh_1.00u" (id 2) (at 102.235 142.875 0)
+    (property "Footprint" "Switch_Keyboard_Kailh:SW_Hotswap_Kailh_1.25u" (id 2) (at 102.235 142.875 0)
       (effects (font (size 1.524 1.524)) hide)
     )
@@
       (effects (font (size 0.508 0.508)))
     )
-    (property "Footprint" "Switch_Keyboard_Kailh:SW_Hotswap_Kailh_1.00u" (id 2) (at 92.075 142.875 0)
+    (property "Footprint" "Switch_Keyboard_Kailh:SW_Hotswap_Kailh_1.25u" (id 2) (at 92.075 142.875 0)
       (effects (font (size 1.524 1.524)) hide)
     )
@@
       (effects (font (size 0.508 0.508)))
     )
-    (property "Footprint" "Switch_Keyboard_Kailh:SW_Hotswap_Kailh_1.00u" (id 2) (at 92.075 126.365 0)
+    (property "Footprint" "Switch_Keyboard_Kailh:SW_Hotswap_Kailh_2.25u" (id 2) (at 92.075 126.365 0)
       (effects (font (size 1.524 1.524)) hide)
     )
@@
       (effects (font (size 0.508 0.508)))
     )
-    (property "Footprint" "Switch_Keyboard_Kailh:SW_Hotswap_Kailh_1.00u" (id 2) (at 202.565 126.365 0)
+    (property "Footprint" "Switch_Keyboard_Kailh:SW_Hotswap_Kailh_1.75u" (id 2) (at 202.565 126.365 0)
       (effects (font (size 1.524 1.524)) hide)
     )
@@
       (effects (font (size 0.508 0.508)))
     )
-    (property "Footprint" "Switch_Keyboard_Kailh:SW_Hotswap_Kailh_1.00u" (id 2) (at 142.875 142.875 0)
+    (property "Footprint" "Switch_Keyboard_Kailh:SW_Hotswap_Kailh_6.25u" (id 2) (at 142.875 142.875 0)
       (effects (font (size 1.524 1.524)) hide)
     )
@@
       (effects (font (size 0.508 0.508)))
     )
-    (property "Footprint" "Switch_Keyboard_Kailh:SW_Hotswap_Kailh_1.00u" (id 2) (at 222.885 76.835 0)
+    (property "Footprint" "Switch_Keyboard_Kailh:SW_Hotswap_Kailh_2.00u" (id 2) (at 222.885 76.835 0)
       (effects (font (size 1.524 1.524)) hide)
     )
@@
       (effects (font (size 0.508 0.508)))
     )
-    (property "Footprint" "Switch_Keyboard_Kailh:SW_Hotswap_Kailh_1.00u" (id 2) (at 112.395 142.875 0)
+    (property "Footprint" "Switch_Keyboard_Kailh:SW_Hotswap_Kailh_1.25u" (id 2) (at 112.395 142.875 0)
       (effects (font (size 1.524 1.524)) hide)
     )
@@
       (effects (font (size 0.508 0.508)))
     )
-    (property "Footprint" "Switch_Keyboard_Kailh:SW_Hotswap_Kailh_1.00u" (id 2) (at 222.885 93.345 0)
+    (property "Footprint" "Switch_Keyboard_Kailh:SW_Hotswap_Kailh_1.50u" (id 2) (at 222.885 93.345 0)
       (effects (font (size 1.524 1.524)) hide)
     )
@@
       (effects (font (size 0.508 0.508)))
     )
-    (property "Footprint" "Switch_Keyboard_Kailh:SW_Hotswap_Kailh_1.00u" (id 2) (at 212.725 109.855 0)
+    (property "Footprint" "Switch_Keyboard_Kailh:SW_Hotswap_Kailh_2.25u" (id 2) (at 212.725 109.855 0)
       (effects (font (size 1.524 1.524)) hide)
     )
@@
     )
     (path "/9fc0a1ee-90cf-486a-8fec-111bf8a1f3e4"
-      (reference "ALT1") (unit 1) (value "MX-NoLED") (footprint "Switch_Keyboard_Kailh:SW_Hotswap_Kailh_1.00u")
+      (reference "ALT1") (unit 1) (value "MX-NoLED") (footprint "Switch_Keyboard_Kailh:SW_Hotswap_Kailh_1.25u")
     )
     (path "/f388a10b-e825-4f38-a6be-0e1b25191ab2"
@@
     )
     (path "/95ebae54-2d90-47e3-aab5-b2e2386ee8be"
-      (reference "BACK1") (unit 1) (value "MX-NoLED") (footprint "Switch_Keyboard_Kailh:SW_Hotswap_Kailh_1.00u")
+      (reference "BACK1") (unit 1) (value "MX-NoLED") (footprint "Switch_Keyboard_Kailh:SW_Hotswap_Kailh_2.00u")
     )
     (path "/3e1718d6-0ef3-41c5-abc0-b80b8834a184"
@@
     )
     (path "/72a2d549-5785-4297-bb09-48200a8916ff"
-      (reference "CAPS1") (unit 1) (value "MX-NoLED") (footprint "Switch_Keyboard_Kailh:SW_Hotswap_Kailh_1.00u")
+      (reference "CAPS1") (unit 1) (value "MX-NoLED") (footprint "Switch_Keyboard_Kailh:SW_Hotswap_Kailh_1.75u")
     )
     (path "/7769c248-1ed9-4dbd-aa80-27946f82ea9b"
-      (reference "CLT1") (unit 1) (value "MX-NoLED") (footprint "Switch_Keyboard_Kailh:SW_Hotswap_Kailh_1.00u")
+      (reference "CLT1") (unit 1) (value "MX-NoLED") (footprint "Switch_Keyboard_Kailh:SW_Hotswap_Kailh_1.25u")
     )
     (path "/fcb9861f-3c51-4a66-ac0f-700eaf2044d5"
@@
     )
     (path "/c9cbc253-e148-4180-a3f9-ce7ef02ca843"
-      (reference "ENTER1") (unit 1) (value "MX-NoLED") (footprint "Switch_Keyboard_Kailh:SW_Hotswap_Kailh_1.00u")
+      (reference "ENTER1") (unit 1) (value "MX-NoLED") (footprint "Switch_Keyboard_Kailh:SW_Hotswap_Kailh_2.25u")
     )
     (path "/b0b4366c-fd02-4020-9d99-38d4220e3979"
@@
     )
     (path "/796e5ad7-8c8a-4e18-85ad-50e9ca8328df"
-      (reference "L_SHIFT1") (unit 1) (value "MX-NoLED") (footprint "Switch_Keyboard_Kailh:SW_Hotswap_Kailh_1.00u")
+      (reference "L_SHIFT1") (unit 1) (value "MX-NoLED") (footprint "Switch_Keyboard_Kailh:SW_Hotswap_Kailh_2.25u")
     )
     (path "/28f82a0f-6cc1-475c-89e6-d9cac169199d"
@@
     )
     (path "/909d6aa5-bb36-41f5-8ba9-9636f6763f73"
-      (reference "R_SHIFT1") (unit 1) (value "MX-NoLED") (footprint "Switch_Keyboard_Kailh:SW_Hotswap_Kailh_1.00u")
+      (reference "R_SHIFT1") (unit 1) (value "MX-NoLED") (footprint "Switch_Keyboard_Kailh:SW_Hotswap_Kailh_1.75u")
     )
     (path "/708715e5-af7d-4bf8-a675-5c0459a272ca"
@@
     )
     (path "/95d732dc-de3b-4a45-b6f1-a124d737cc28"
-      (reference "SPACE1") (unit 1) (value "MX-NoLED") (footprint "Switch_Keyboard_Kailh:SW_Hotswap_Kailh_1.00u")
+      (reference "SPACE1") (unit 1) (value "MX-NoLED") (footprint "Switch_Keyboard_Kailh:SW_Hotswap_Kailh_6.25u")
     )
     (path "/7358fe96-0654-4f3a-a506-932be01f6f97"
@@
     )
     (path "/39ca259b-b6f2-465e-bf01-26d2c0a47907"
-      (reference "TAB1") (unit 1) (value "MX-NoLED") (footprint "Switch_Keyboard_Kailh:SW_Hotswap_Kailh_1.00u")
+      (reference "TAB1") (unit 1) (value "MX-NoLED") (footprint "Switch_Keyboard_Kailh:SW_Hotswap_Kailh_1.50u")
     )
     (path "/1de20f08-09dc-4bca-bd53-e579edc44b85"
@@
     )
     (path "/750a78d2-5a83-4d1a-bea9-155d09db2d56"
-      (reference "WIN1") (unit 1) (value "MX-NoLED") (footprint "Switch_Keyboard_Kailh:SW_Hotswap_Kailh_1.00u")
+      (reference "WIN1") (unit 1) (value "MX-NoLED") (footprint "Switch_Keyboard_Kailh:SW_Hotswap_Kailh_1.25u")
     )
     (path "/9a29e96a-1893-4403-b940-72a573b2f934"
@@
     )
     (path "/a8c76cdf-6ef1-4b7e-8eb8-32559e1891b9"
-      (reference "\\1") (unit 1) (value "MX-NoLED") (footprint "Switch_Keyboard_Kailh:SW_Hotswap_Kailh_1.00u")
+      (reference "\\1") (unit 1) (value "MX-NoLED") (footprint "Switch_Keyboard_Kailh:SW_Hotswap_Kailh_1.50u")
     )
     (path "/20b7abac-571e-4459-b421-17207a6f4ca5"

Commit message: routing pcb
Parts:
- added C2, C3: 22pF, Capacitor_SMD:C_0603_1608Metric, symbol Device:C_Small
- added C4, C5, C6, C7: 0.1uF, Capacitor_SMD:C_0603_1608Metric, symbol Device:C_Small
- added C8: 100uF, Capacitor_SMD:C_0603_1608Metric, symbol Device:C_Small
- added R2, R5: 10k, Resistor_SMD:R_0603_1608Metric, symbol Device:R
- added R3, R4: 22, Resistor_SMD:R_0603_1608Metric, symbol Device:R
- added SW1: RotaryEncoder_Switch, Rotary_Encoder:RotaryEncoder_Alps_EC11E-Switch_Vertical_H20mm, symbol Device:RotaryEncoder_Switch
- added U2: ATmega32U4-A, Package_QFP:TQFP-44_10x10mm_P0.8mm, symbol MCU_Microchip_ATmega:ATmega32U4-A
- added Y2: Crystal_GND24_Small, Crystal:Crystal_SMD_3225-4Pin_3.2x2.5mm, symbol Device:Crystal_GND24_Small
- D1, D10, D11, D12, D13, D14, D15, D16, D17, D18, D19, D2, D20, D21, D22, D23, D24, D25, D26, D27, D28, D29, D3, D30, D31, D32, D33, D34, D35, D36, D37, D38, D39, D4, D40, D41, D42, D43, D44, D45, D47, D48, D49, D5, D50, D51, D52, D53, D54, D55, D56, D57, D58, D59, D6, D60, D61, D62, D63, D64, D65, D66, D67, D68, D69, D7, D70, D71, D72, D73, D74, D75, D76, D77, D78, D79, D8, D80, D81, D82, D83, D84, D9: footprint Diode_SMD:D_0603_1608Metric_Pad1.05x0.95mm_HandSolder -> Diode_SMD:D_SOD-123
Connections:
- net ROW5: now reaches D61.1 (K), D62.1 (K), D63.1 (K), D64.1 (K), D65.1 (K), D66.1 (K), D67.1 (K), D68.1 (K), D69.1 (K), D70.1 (K), D71.1 (K), D72.1 (K), D73.1 (K), D74.1 (K)
- net ROW5: now also U2.29 (PB5)
- net COL11: now reaches /1.1 (COL), ;1.1 (COL), F10.1 (COL), FN1.1 (COL), MX10.1 (COL), P1.1 (COL)
- net COL11: now also U2.37 (PF6)
- net COL12: now reaches '1.1 (COL), -1.1 (COL), CTL1.1 (COL), F11.1 (COL), R_SHIFT1.1 (COL), [1.1 (COL)
- net COL12: now also U2.38 (PF5)
- net ROW3: now reaches D31.1 (K), D32.1 (K), D33.1 (K), D34.1 (K), D35.1 (K), D36.1 (K), D37.1 (K), D38.1 (K), D39.1 (K), D40.1 (K), D41.1 (K), D42.1 (K), D43.1 (K), D44.1 (K), D45.1 (K)
- net ROW3: now also U2.31 (PC6)
- net COL10: now reaches .1.1 (COL), ALT2.1 (COL), F9.1 (COL), L1.1 (COL), MX9.1 (COL), O1.1 (COL)
- net COL10: now also U2.36 (PF7)
- net ROW4: now reaches D47.1 (K), D48.1 (K), D49.1 (K), D50.1 (K), D51.1 (K), D52.1 (K), D53.1 (K), D54.1 (K), D55.1 (K), D56.1 (K), D57.1 (K), D58.1 (K), D59.1 (K), D60.1 (K)
- net ROW4: now also U2.30 (PB6)
- net COL15: now reaches OPT1.1 (COL), OPT2.1 (COL), OPT3.1 (COL), OPT4.1 (COL), OPT5.1 (COL), RIGHT1.1 (COL)
- net COL15: now also SW1.S1, U2.41 (PF0)
- net ROT1: now reaches D15.2 (A), OPT1.2 (ROW)
- net ROT1: now also SW1.S2
- net ROW1: now reaches D1.1 (K), D10.1 (K), D11.1 (K), D12.1 (K), D13.1 (K), D14.1 (K), D15.1 (K), D2.1 (K), D3.1 (K), D4.1 (K), D5.1 (K), D6.1 (K), D7.1 (K), D8.1 (K), D9.1 (K)
- net ROW2: now reaches D16.1 (K), D17.1 (K), D18.1 (K), D19.1 (K), D20.1 (K), D21.1 (K), D22.1 (K), D23.1 (K), D24.1 (K), D25.1 (K), D26.1 (K), D27.1 (K), D28.1 (K), D29.1 (K), D30.1 (K)
- net ROW2: now also U2.32 (PC7)
- net COL8: now reaches F7.1 (COL), J1.1 (COL), M1.1 (COL), MX7.1 (COL), U1.1 (COL)
- net COL8: now also U2.26 (PD6)
- net COL13: now reaches +1.1 (COL), ENTER1.1 (COL), F12.1 (COL), LEFT1.1 (COL), ]1.1 (COL)
- net COL13: now also U2.39 (PF4)
- net COL9: now reaches ,1.1 (COL), F8.1 (COL), I1.1 (COL), K1.1 (COL), MX8.1 (COL)
- net COL9: now also U2.27 (PD7)
- net COL14: now reaches BACK1.1 (COL), DEL1.1 (COL), DOWN1.1 (COL), UP1.1 (COL), \1.1 (COL)
- net COL14: now also U2.40 (PF1)
- net COL1: now reaches CAPS1.1 (COL), CLT1.1 (COL), L_SHIFT1.1 (COL), TAB1.1 (COL), `~1.1 (COL), esc1.1 (COL)
- net COL1: now also U2.12 (PB7)
- net COL4: now reaches C1.1 (COL), D46.1 (COL), E1.1 (COL), F3.1 (COL), MX3.1 (COL)
- net COL4: now also U2.20 (PD2)
- net ROW6: now reaches D75.1 (K), D76.1 (K), D77.1 (K), D78.1 (K), D79.1 (K), D80.1 (K), D81.1 (K), D82.1 (K), D83.1 (K), D84.1 (K)
- net ROW6: now also U2.28 (PB4)
- net COL2: now reaches A1.1 (COL), F1.1 (COL), MX1.1 (COL), Q1.1 (COL), WIN1.1 (COL), Z1.1 (COL)
- net COL2: now also U2.18 (PD0)
- net COL6: now reaches B1.1 (COL), F5.1 (COL), G1.1 (COL), MX5.1 (COL), SPACE1.1 (COL), T1.1 (COL)
- net COL6: now also U2.22 (PD5)
- net COL3: now reaches ALT1.1 (COL), F2.1 (COL), MX2.1 (COL), S1.1 (COL), W1.1 (COL), X1.1 (COL)
- net COL3: now also U2.19 (PD1)
- net COL5: now reaches F13.1 (COL), F4.1 (COL), MX4.1 (COL), R1.1 (COL), V1.1 (COL)
- net COL5: now also U2.21 (PD3)
- net COL7: now reaches F6.1 (COL), H1.1 (COL), MX6.1 (COL), N1.1 (COL), Y1.1 (COL)
- net COL7: now also U2.25 (PD4)
- new net: R5.1, U2.33 (~{HWB}/PE2)
- new net: R4.2, U2.3 (D-)
- new net: C4.1, U2.6 (UCAP)
- new net: R2.2, U2.13 (~{RESET})
- new net: C2.1, U2.17 (XTAL1), Y2.3
- new net: C3.2, U2.16 (XTAL2), Y2.1
- new net: R3.1, U2.4 (D+)
- new net +5V: C5.1, C6.1, C7.1, C8.1, R2.1, U2.14 (VCC), U2.2 (UVCC), U2.24 (AVCC), U2.34 (VCC), U2.44 (AVCC), U2.7 (VBUS)
- new net D+: R3.2
- new net D-: R4.1
- new net GND: C2.2, C3.1, C4.2, C5.2, C6.2, C7.2, C8.2, R5.2, SW1.C, U2.15 (GND), U2.23 (GND), U2.35 (GND), U2.43 (GND), U2.5 (UGND), Y2.2, Y2.4
- new net ROT_A: SW1.A, U2.9 (PB1)
- new net ROT_B: SW1.B, U2.8 (PB0)
Other:
- moved on the sheet: '1, +1, ,1, -1, .1, /1, ;1, A1, ALT1, ALT2, B1, BACK1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
