File: fese75.kicad_sch (KiCad schematic)
At the start: 205 parts, among them J1 MX-NoLED, J2 USB_C_Receptacle_USB2.0, K1 MX-NoLED, M1 MX-NoLED, P1 MX-NoLED, Q1 MX-NoLED, SW1 RotaryEncoder_Switch, T1 MX-NoLED, U1 MX-NoLED, U2 ATmega32U4-A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

Commit message: change distant from 0.5 to 0.25
Parts:
- removed TP10: CO8, TestPoint:TestPoint_THTPad_D2.0mm_Drill1.0mm, symbol Connector:TestPoint
- removed TP11: CO9, TestPoint:TestPoint_THTPad_D2.0mm_Drill1.0mm, symbol Connector:TestPoint
- removed TP12: CO10, TestPoint:TestPoint_THTPad_D2.0mm_Drill1.0mm, symbol Connector:TestPoint
- removed TP13: CO11, TestPoint:TestPoint_THTPad_D2.0mm_Drill1.0mm, symbol Connector:TestPoint
- removed TP14: CO12, TestPoint:TestPoint_THTPad_D2.0mm_Drill1.0mm, symbol Connector:TestPoint
- removed TP15: CO13, TestPoint:TestPoint_THTPad_D2.0mm_Drill1.0mm, symbol Connector:TestPoint
- removed TP16: CO14, TestPoint:TestPoint_THTPad_D2.0mm_Drill1.0mm, symbol Connector:TestPoint
- removed TP17: CO15, TestPoint:TestPoint_THTPad_D2.0mm_Drill1.0mm, symbol Connector:TestPoint
- removed TP18: RO1, TestPoint:TestPoint_THTPad_2.0x2.0mm_Drill1.0mm, symbol Connector:TestPoint
- removed TP19: RO2, TestPoint:TestPoint_THTPad_D2.0mm_Drill1.0mm, symbol Connector:TestPoint
- removed TP20: RO3, TestPoint:TestPoint_THTPad_D2.0mm_Drill1.0mm, symbol Connector:TestPoint
- removed TP21: RO4, TestPoint:TestPoint_THTPad_D2.0mm_Drill1.0mm, symbol Connector:TestPoint
- removed TP22: RO5, TestPoint:TestPoint_THTPad_D2.0mm_Drill1.0mm, symbol Connector:TestPoint
- removed TP23: RO6, TestPoint:TestPoint_THTPad_D2.0mm_Drill1.0mm, symbol Connector:TestPoint
- removed TP3: CO1, TestPoint:TestPoint_THTPad_2.0x2.0mm_Drill1.0mm, symbol Connector:TestPoint
- removed TP4: CO2, TestPoint:TestPoint_THTPad_D2.0mm_Drill1.0mm, symbol Connector:TestPoint
- removed TP5: CO3, TestPoint:TestPoint_THTPad_D2.0mm_Drill1.0mm, symbol Connector:TestPoint
- removed TP6: CO4, TestPoint:TestPoint_THTPad_D2.0mm_Drill1.0mm, symbol Connector:TestPoint
- removed TP7: CO5, TestPoint:TestPoint_THTPad_D2.0mm_Drill1.0mm, symbol Connector:TestPoint
- removed TP8: CO6, TestPoint:TestPoint_THTPad_D2.0mm_Drill1.0mm, symbol Connector:TestPoint
- removed TP9: CO7, TestPoint:TestPoint_THTPad_D2.0mm_Drill1.0mm, symbol Connector:TestPoint
- added J3: Conn_01x15_Female, Connector_PinHeader_2.54mm:PinHeader_1x15_P2.54mm_Vertical, symbol Connector:Conn_01x15_Female
- added J4: Conn_01x06_Female, Connector_PinHeader_2.54mm:PinHeader_1x06_P2.54mm_Vertical, symbol Connector:Conn_01x06_Female
Connections:
- net COL1: now also J3.1 (Pin_1)
- net COL10: now also J3.10 (Pin_10)
- net COL11: now also J3.11 (Pin_11)
- net COL12: now also J3.12 (Pin_12)
- net COL13: now also J3.13 (Pin_13)
- net COL14: now also J3.14 (Pin_14)
- net COL15: now also J3.15 (Pin_15)
- net COL2: now also J3.2 (Pin_2)
- net COL3: now also J3.3 (Pin_3)
- net COL4: now also J3.4 (Pin_4)
- net COL5: now also J3.5 (Pin_5)
- net COL6: now also J3.6 (Pin_6)
- net COL7: now also J3.7 (Pin_7)
- net COL8: now also J3.8 (Pin_8)
- net COL9: now also J3.9 (Pin_9)
- net ROW1: now also J4.1 (Pin_1)
- net ROW2: now also J4.2 (Pin_2)
- net ROW3: now also J4.3 (Pin_3)
- net ROW4: now also J4.4 (Pin_4)
- net ROW5: now also J4.5 (Pin_5)
- net ROW6: now also J4.6 (Pin_6)
