File: _autosave-fese75.kicad_pcb (KiCad board)
At the start: 2 copper layers, 319.1 x 133.3 mm, 190 parts, among them J1 MX-NoLED, J2 USB_C_Receptacle_USB2.0, J3 Conn_01x15_Male, J4 Conn_01x06_Female, K1 MX-NoLED, M1 MX-NoLED, P1 MX-NoLED, Q1 MX-NoLED, SW1 RotaryEncoder_Switch, T1 MX-NoLED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

Commit message: change distant from 0.5 to 0.25
Parts:
- moved D1 4.76 mm to (50.8, 65.1)
- moved D10 4.76 mm to (236.6, 65.1)
- moved D11 4.76 mm to (255.7, 65.1)
- moved D12 4.76 mm to (274.7, 65.1)
- moved D13 4.76 mm to (293.8, 65.1)
- moved D14 4.76 mm to (317.6, 65.1)
- moved D15 4.76 mm to (346.1, 65.1)
- moved D2 4.76 mm to (74.7, 65.2)
- moved D3 4.76 mm to (93.8, 65.1)
- moved D4 4.76 mm to (112.8, 65.1)
- moved D5 4.76 mm to (132.0, 65.1)
- moved D6 4.76 mm to (155.6, 65.1)
- moved D7 4.76 mm to (174.7, 65.1)
- moved D8 4.76 mm to (193.8, 65.1)
- moved D9 4.76 mm to (212.9, 65.1)
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Routing:
- net COL14: track 442.8 -> 415.0 mm
- net COL1: track 411.7 -> 404.2 mm
- net COL2: track 375.2 -> 368.3 mm
- net COL8: track 128.4 -> 122.8 mm
- net VCC: track 209.1 -> 204.3 mm
- net D+: track 237.5 -> 232.7 mm
- net GND: track 326.0 -> 321.2 mm
- net D-: track 236.9 -> 232.2 mm
- net ROT_A: track 256.5 -> 251.8 mm
- net ROT_B: track 257.9 -> 253.2 mm
- net ROW1: track 667.3 -> 662.6 mm
- net COL7: track 166.2 -> 162.2 mm
- net COL5: track 280.8 -> 276.7 mm
- net COL4: track 331.8 -> 327.8 mm
- net COL3: track 407.5 -> 403.4 mm
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Other:
- board size 319.1 x 133.3 mm -> 319.1 x 128.6 mm
